Commit message: modify urdf files

File: urdf/kr300r2500ultra.urdf (robot description, URDF)
Before this commit: robot kuka_kr300r2500ultra, 9 links, 8 joints
Joints:
- joint joint_a1: limit lower=-3.2288591161895095 upper=3.2288591161895095 effort=0 velocity=2.722713633111154 -> lower=-0.05635422266054108 upper=0.05635422266054108 effort=0 velocity=0.047520317486726533
- joint joint_a2: limit lower=-2.705260340591211 upper=0.6108652381980153 effort=0 velocity=2.722713633111154 -> lower=-0.04721570006693983 upper=0.0106616096925348 effort=0 velocity=0.047520317486726533
- joint joint_a3: limit lower=-2.2689280275926285 upper=2.6878070480712677 effort=0 velocity=2.722713633111154 -> lower=-0.039600264572272115 upper=0.04691108264715312 effort=0 velocity=0.047520317486726533; origin xyz=1.150 0 0 rpy=0 0 0 -> xyz=1.15 0 0 rpy=0 0 0
- joint joint_a4: limit lower=-6.1086523819801535 upper=6.1086523819801535 effort=0 velocity=5.759586531581287 -> lower=-0.10661609692534801 upper=0.10661609692534801 effort=0 velocity=0.10052374852961382
- joint joint_a5: limit lower=-2.2689280275926285 upper=2.2689280275926285 effort=0 velocity=5.759586531581287 -> lower=-0.039600264572272115 upper=0.039600264572272115 effort=0 velocity=0.10052374852961382
- joint joint_a6: limit lower=-6.1086523819801535 upper=6.1086523819801535 effort=0 velocity=10.733774899765127 -> lower=-0.10661609692534801 upper=0.10661609692534801 effort=0 velocity=0.18733971316882578
- joint joint_a6-tool0: origin xyz=0.240 0 0 rpy=0 1.5707963267948966 0 -> xyz=0.24 0 0 rpy=0 1.5707963267948966 0

File: urdf/kr300r2500ultra.xacro (robot description, xacro)
@@ -1,3 +1,7 @@
 <?xml version="1.0"?>
+<!-- =================================================================================== -->
+<!-- |    This document was autogenerated by xacro from kr300r2500ultra.xacro            | -->
+<!-- |    EDITING THIS FILE BY HAND IS NOT RECOMMENDED                                 | -->
+<!-- =================================================================================== -->
 <!--Generates a urdf from the macro in kr300r2500ultra_macro.xacro -->
 <robot name="kuka_kr300r2500ultra" xmlns:xacro="http://wiki.ros.org/xacro">

File: urdf/kr300r2500ultra_macro.xacro (robot description, xacro)
@@ -2,4 +2,7 @@
 <robot xmlns:xacro="http://wiki.ros.org/xacro">
   <xacro:property name="DEG2RAD" value="0.017453292519943295"/>
+  <!-- Load configuration files -->
+  <xacro:property name="kinematics" value="${load_yaml('$(find kuka_kr300_support)/config/default_kinematics.yaml')}"/>
+  <xacro:property name="joint_limits" value="${load_yaml('$(find kuka_kr300_support)/config/joint_limits.yaml')}"/>
   <xacro:macro name="kuka_kr300r2500ultra" params="prefix">
     <!-- LINKS -->
@@ -172,55 +175,80 @@
     <!-- joint 1 (A1) -->
     <joint name="${prefix}joint_a1" type="revolute">
-      <origin xyz="0 0 0.675" rpy="0 0 0"/>
+      <origin xyz="${kinematics['kinematics']['joint_a1']['x']} ${kinematics['kinematics']['joint_a1']['y']} ${kinematics['kinematics']['joint_a1']['z']}"
+              rpy="${kinematics['kinematics']['joint_a1']['roll']} ${kinematics['kinematics']['joint_a1']['pitch']} ${kinematics['kinematics']['joint_a1']['yaw']}"/>
       <parent link="${prefix}base_link"/>
       <child link="${prefix}link_1"/>
       <axis xyz="0 0 -1"/>
-      <limit effort="0" lower="${-DEG2RAD * 185}" upper="${DEG2RAD * 185}" velocity="${DEG2RAD * 156}"/>
+      <limit effort="${joint_limits['joint_limits']['joint_a1']['max_effort']}"
+             lower="${DEG2RAD * joint_limits['joint_limits']['joint_a1']['min_position']}"
+             upper="${DEG2RAD * joint_limits['joint_limits']['joint_a1']['max_position']}"
+             velocity="${DEG2RAD * joint_limits['joint_limits']['joint_a1']['max_velocity']}"/>
     </joint>
     <!-- joint 2 (A2) -->
     <joint name="${prefix}joint_a2" type="revolute">
-      <origin xyz="0.35 0 0" rpy="0 0 0"/>
+      <origin xyz="${kinematics['kinematics']['joint_a2']['x']} ${kinematics['kinematics']['joint_a2']['y']} ${kinematics['kinematics']['joint_a2']['z']}"
+              rpy="${kinematics['kinematics']['joint_a2']['roll']} ${kinematics['kinematics']['joint_a2']['pitch']} ${kinematics['kinematics']['joint_a2']['yaw']}"/>
       <parent link="${prefix}link_1"/>
       <child link="${prefix}link_2"/>
       <axis xyz="0 1 0"/>
-      <limit effort="0" lower="${-DEG2RAD * 155}" upper="${DEG2RAD * 35}" velocity="${DEG2RAD * 156}"/>
+      <limit effort="${joint_limits['joint_limits']['joint_a2']['max_effort']}"
+             lower="${DEG2RAD * joint_limits['joint_limits']['joint_a2']['min_position']}"
+             upper="${DEG2RAD * joint_limits['joint_limits']['joint_a2']['max_position']}"
+             velocity="${DEG2RAD * joint_limits['joint_limits']['joint_a2']['max_velocity']}"/>
     </joint>
     <!-- joint 3 (A3) -->
     <joint name="${prefix}joint_a3" type="revolute">
-      <origin xyz="1.150 0 0" rpy="0 0 0"/>
+      <origin xyz="${kinematics['kinematics']['joint_a3']['x']} ${kinematics['kinematics']['joint_a3']['y']} ${kinematics['kinematics']['joint_a3']['z']}"
+              rpy="${kinematics['kinematics']['joint_a3']['roll']} ${kinematics['kinematics']['joint_a3']['pitch']} ${kinematics['kinematics']['joint_a3']['yaw']}"/>
       <parent link="${prefix}link_2"/>
       <child link="${prefix}link_3"/>
       <axis xyz="0 1 0"/>
-      <limit effort="0" lower="${-DEG2RAD * 130}" upper="${DEG2RAD * 154}" velocity="${DEG2RAD * 156}"/>
+      <limit effort="${joint_limits['joint_limits']['joint_a3']['max_effort']}"
+             lower="${DEG2RAD * joint_limits['joint_limits']['joint_a3']['min_position']}"
+             upper="${DEG2RAD * joint_limits['joint_limits']['joint_a3']['max_position']}"
+             velocity="${DEG2RAD * joint_limits['joint_limits']['joint_a3']['max_velocity']}"/>
     </joint>
     <!-- joint 4 (A4) -->
     <joint name="${prefix}joint_a4" type="revolute">
-      <origin xyz="1.0 0 -0.041" rpy="0 0 0"/>
+      <origin xyz="${kinematics['kinematics']['joint_a4']['x']} ${kinematics['kinematics']['joint_a4']['y']} ${kinematics['kinematics']['joint_a4']['z']}"
+              rpy="${kinematics['kinematics']['joint_a4']['roll']} ${kinematics['kinematics']['joint_a4']['pitch']} ${kinematics['kinematics']['joint_a4']['yaw']}"/>
       <parent link="${prefix}link_3"/>
       <child link="${prefix}link_4"/>
       <axis xyz="-1 0 0"/>
-      <limit effort="0" lower="${-DEG2RAD * 350}" upper="${DEG2RAD * 350}" velocity="${DEG2RAD * 330}"/>
+      <limit effort="${joint_limits['joint_limits']['joint_a4']['max_effort']}"
+             lower="${DEG2RAD * joint_limits['joint_limits']['joint_a4']['min_position']}"
+             upper="${DEG2RAD * joint_limits['joint_limits']['joint_a4']['max_position']}"
+             velocity="${DEG2RAD * joint_limits['joint_limits']['joint_a4']['max_velocity']}"/>
     </joint>
     <!-- joint 5 (A5) -->
     <joint name="${prefix}joint_a5" type="revolute">
-      <origin xyz="0 0 0" rpy="0 0 0"/>
+      <origin xyz="${kinematics['kinematics']['joint_a5']['x']} ${kinematics['kinematics']['joint_a5']['y']} ${kinematics['kinematics']['joint_a5']['z']}"
+              rpy="${kinematics['kinematics']['joint_a5']['roll']} ${kinematics['kinematics']['joint_a5']['pitch']} ${kinematics['kinematics']['joint_a5']['yaw']}"/>
       <parent link="${prefix}link_4"/>
       <child link="${prefix}link_5"/>
       <axis xyz="0 1 0"/>
-      <limit effort="0" lower="${-DEG2RAD * 130}" upper="${DEG2RAD * 130}" velocity="${DEG2RAD * 330}"/>
+      <limit effort="${joint_limits['joint_limits']['joint_a5']['max_effort']}"
+             lower="${DEG2RAD * joint_limits['joint_limits']['joint_a5']['min_position']}"
+             upper="${DEG2RAD * joint_limits['joint_limits']['joint_a5']['max_position']}"
+             velocity="${DEG2RAD * joint_limits['joint_limits']['joint_a5']['max_velocity']}"/>
     </joint>
     <!-- joint 6 (A6) -->
     <joint name="${prefix}joint_a6" type="revolute">
-      <origin xyz="0 0 0" rpy="0 0 0"/>
+      <origin xyz="${kinematics['kinematics']['joint_a6']['x']} ${kinematics['kinematics']['joint_a6']['y']} ${kinematics['kinematics']['joint_a6']['z']}"
+              rpy="${kinematics['kinematics']['joint_a6']['roll']} ${kinematics['kinematics']['joint_a6']['pitch']} ${kinematics['kinematics']['joint_a6']['yaw']}"/>
       <parent link="${prefix}link_5"/>
       <child link="${prefix}link_6"/>
       <axis xyz="-1 0 0"/>
-      <limit effort="0" lower="${-DEG2RAD * 350}" upper="${DEG2RAD * 350}" velocity="${DEG2RAD * 615}"/>
+      <limit effort="${joint_limits['joint_limits']['joint_a6']['max_effort']}"
+             lower="${DEG2RAD * joint_limits['joint_limits']['joint_a6']['min_position']}"
+             upper="${DEG2RAD * joint_limits['joint_limits']['joint_a6']['max_position']}"
+             velocity="${DEG2RAD * joint_limits['joint_limits']['joint_a6']['max_velocity']}"/>
     </joint>
     <!-- tool frame - fixed frame -->
     <joint name="${prefix}joint_a6-tool0" type="fixed">
+      <origin xyz="${kinematics['kinematics']['joint_a6-tool0']['x']} ${kinematics['kinematics']['joint_a6-tool0']['y']} ${kinematics['kinematics']['joint_a6-tool0']['z']}"
+              rpy="${kinematics['kinematics']['joint_a6-tool0']['roll']} ${kinematics['kinematics']['joint_a6-tool0']['pitch']} ${kinematics['kinematics']['joint_a6-tool0']['yaw']}"/>
       <parent link="${prefix}link_6"/>
       <child link="${prefix}tool0"/>
-      <origin xyz="0.240 0 0" rpy="0 ${DEG2RAD * 90} 0"/>
     </joint>
     <!-- END JOINTS -->
